File: cpu-sheet.kicad_sch (KiCad schematic)
At the start: 53 parts, among them J3 GPIO_HEADER, J4 GPIOR_HEADER, J5 USB_B_Micro, J6 PROG_CONN, U11 CH340G, U6 SRV05-4, U7 23LC1024, U8 STM32L432KC, U9 SRV05-4, Y2 32.768K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

Commit message: added PWRLED, both headers now 6-pin. DRC ok. TODO list empty.
Parts:
- added R91: 330, Resistor_SMD:R_0603_1608Metric, symbol Device:R_Small
- J3, J4: footprint Connector_PinHeader_2.54mm:PinHeader_1x05_P2.54mm_Vertical_SMD_Pin1Left -> Connector_PinHeader_2.54mm:PinHeader_1x06_P2.54mm_Vertical_SMD_Pin1Left; symbol Connector:Conn_01x05_Male -> Connector:Conn_01x06_Male; LCSC C780063 -> C5160789
Connections:
- net 3V8_OUT: now also J3.6 (Pin_6); no longer J3.5 (Pin_5)
- net GND: now also J3.2 (Pin_2), J3.5 (Pin_5), J4.6 (Pin_6); no longer J3.4 (Pin_4), J4.5 (Pin_5)
- net GPIO10_TERMINAL: now also J3.4 (Pin_4); no longer J3.3 (Pin_3)
- net GPIO11_TERMINAL: now also J3.3 (Pin_3); no longer J3.2 (Pin_2)
- net GPIOR1: now also J4.2 (Pin_2); no longer J4.1 (Pin_1)
- net GPIOR2: now also J4.3 (Pin_3); no longer J4.2 (Pin_2)
- net at C54.2, R26.2: now also J4.5 (Pin_5); no longer J4.4 (Pin_4)
- net at R45.2: now also J4.4 (Pin_4); no longer J4.3 (Pin_3)
- new net: J4.1 (Pin_1), R91.2
- new net 3V3_LNA: R91.1
