File: linreg-sheet.kicad_sch (KiCad schematic)
At the start: 20 parts, among them J1 PWR_TERM, J2 PWR_TERM, U12 XC6206PxxxMR, U13 XC6206PxxxMR, U16 XC6206PxxxMR, U4 XC6206PxxxMR

Commit message: misc
Changed lines of the file:
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@@
     (stroke (width 0) (type default) (color 0 0 0 0))
   )
-  (text "Screw terminals" (at 72.39 158.75 0)
+  (text "Screw terminals" (at 63.5 158.75 0)
     (effects (font (size 2.4638 2.4638) (thickness 0.4928) bold) (justify left bottom))
   )
@@
   )
   (global_label "3V8_OUT" (shape input) (at 106.68 35.56 180) (fields_autoplaced)
-    (effects (font (size 2.0066 2.0066)) (justify right))
-    (property "Intersheet References" "${INTERSHEET_REFS}" (id 0) (at 0 0 0)
-      (effects (font (size 1.27 1.27)) hide)
+    (effects (font (size 2.0066 2.0066) (thickness 0.4013) bold) (justify right))
+    (property "Intersheet References" "${INTERSHEET_REFS}" (id 0) (at 89.903 35.3594 0)
+      (effects (font (size 2.0066 2.0066) (thickness 0.4013) bold) (justify right) hide)
     )
   )
   (global_label "3V3_CPU" (shape input) (at 190.5 66.04 0) (fields_autoplaced)
-    (effects (font (size 2.0066 2.0066)) (justify left))
-    (property "Intersheet References" "${INTERSHEET_REFS}" (id 0) (at 0 0 0)
-      (effects (font (size 1.27 1.27)) hide)
+    (effects (font (size 2.0066 2.0066) (thickness 0.4013) bold) (justify left))
+    (property "Intersheet References" "${INTERSHEET_REFS}" (id 0) (at 207.6592 65.8394 0)
+      (effects (font (size 2.0066 2.0066) (thickness 0.4013) bold) (justify left) hide)
     )
   )
   (global_label "3V8_OUT" (shape input) (at 106.68 66.04 180) (fields_autoplaced)
-    (effects (font (size 2.0066 2.0066)) (justify right))
-    (property "Intersheet References" "${INTERSHEET_REFS}" (id 0) (at 0 0 0)
-      (effects (font (size 1.27 1.27)) hide)
+    (effects (font (size 2.0066 2.0066) (thickness 0.4013) bold) (justify right))
+    (property "Intersheet References" "${INTERSHEET_REFS}" (id 0) (at 89.903 65.8394 0)
+      (effects (font (size 2.0066 2.0066) (thickness 0.4013) bold) (justify right) hide)
     )
   )
   (global_label "12V_OUT" (shape input) (at 138.43 172.72 0) (fields_autoplaced)
-    (effects (font (size 2.0066 2.0066)) (justify left))
-    (property "Intersheet References" "${INTERSHEET_REFS}" (id 0) (at 0 0 0)
-      (effects (font (size 1.27 1.27)) hide)
+    (effects (font (size 2.0066 2.0066) (thickness 0.4013) bold) (justify left))
+    (property "Intersheet References" "${INTERSHEET_REFS}" (id 0) (at 155.207 172.5194 0)
+      (effects (font (size 2.0066 2.0066) (thickness 0.4013) bold) (justify left) hide)
     )
   )
   (global_label "3V8_OUT" (shape input) (at 105.41 127 180) (fields_autoplaced)
-    (effects (font (size 2.0066 2.0066)) (justify right))
-    (property "Intersheet References" "${INTERSHEET_REFS}" (id 0) (at 0 0 0)
-      (effects (font (size 1.27 1.27)) hide)
+    (effects (font (size 2.0066 2.0066) (thickness 0.4013) bold) (justify right))
+    (property "Intersheet References" "${INTERSHEET_REFS}" (id 0) (at 88.633 126.7994 0)
+      (effects (font (size 2.0066 2.0066) (thickness 0.4013) bold) (justify right) hide)
     )
   )
   (global_label "3V3_RADIO" (shape input) (at 191.77 97.79 0) (fields_autoplaced)
-    (effects (font (size 2.0066 2.0066)) (justify left))
-    (property "Intersheet References" "${INTERSHEET_REFS}" (id 0) (at 0 0 0)
-      (effects (font (size 1.27 1.27)) hide)
+    (effects (font (size 2.0066 2.0066) (thickness 0.4013) bold) (justify left))
+    (property "Intersheet References" "${INTERSHEET_REFS}" (id 0) (at 211.6047 97.5894 0)
+      (effects (font (size 2.0066 2.0066) (thickness 0.4013) bold) (justify left) hide)
     )
   )
   (global_label "3V3_LNA" (shape input) (at 191.77 127 0) (fields_autoplaced)
-    (effects (font (size 2.0066 2.0066)) (justify left))
-    (property "Intersheet References" "${INTERSHEET_REFS}" (id 0) (at 0 0 0)
-      (effects (font (size 1.27 1.27)) hide)
+    (effects (font (size 2.0066 2.0066) (thickness 0.4013) bold) (justify left))
+    (property "Intersheet References" "${INTERSHEET_REFS}" (id 0) (at 208.2604 126.7994 0)
+      (effects (font (size 2.0066 2.0066) (thickness 0.4013) bold) (justify left) hide)
     )
   )
@@
   )
   (global_label "3V8_OUT" (shape input) (at 105.41 97.79 180) (fields_autoplaced)
-    (effects (font (size 2.0066 2.0066)) (justify right))
-    (property "Intersheet References" "${INTERSHEET_REFS}" (id 0) (at 0 0 0)
-      (effects (font (size 1.27 1.27)) hide)
+    (effects (font (size 2.0066 2.0066) (thickness 0.4013) bold) (justify right))
+    (property "Intersheet References" "${INTERSHEET_REFS}" (id 0) (at 88.633 97.5894 0)
+      (effects (font (size 2.0066 2.0066) (thickness 0.4013) bold) (justify right) hide)
     )
   )
   (global_label "3V3_ETHERNET" (shape input) (at 189.23 35.56 0) (fields_autoplaced)
-    (effects (font (size 2.0066 2.0066)) (justify left))
-    (property "Intersheet References" "${INTERSHEET_REFS}" (id 0) (at 0 0 0)
-      (effects (font (size 1.27 1.27)) hide)
+    (effects (font (size 2.0066 2.0066) (thickness 0.4013) bold) (justify left))
+    (property "Intersheet References" "${INTERSHEET_REFS}" (id 0) (at 214.9889 35.3594 0)
+      (effects (font (size 2.0066 2.0066) (thickness 0.4013) bold) (justify left) hide)
     )
   )

Commit message: added PWRLED, both headers now 6-pin. DRC ok. TODO list empty.
Parts:
- removed TP9: TestPoint, TestPoint:TestPoint_Pad_D1.5mm, symbol Connector:TestPoint
Changed lines of the file:
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@@
   (junction (at 168.91 35.56) (diameter 0) (color 0 0 0 0)
   )
-  (junction (at 111.76 35.56) (diameter 0) (color 0 0 0 0)
-  )
   (junction (at 118.11 127) (diameter 0) (color 0 0 0 0)
   )
@@
     (stroke (width 0) (type default) (color 0 0 0 0))
   )
-  (wire (pts (xy 111.76 35.56) (xy 119.38 35.56))
+  (wire (pts (xy 106.68 35.56) (xy 119.38 35.56))
     (stroke (width 0) (type default) (color 0 0 0 0))
   )
@@
   )
   (wire (pts (xy 156.21 44.45) (xy 156.21 43.18))
-    (stroke (width 0) (type default) (color 0 0 0 0))
-  )
-  (wire (pts (xy 106.68 35.56) (xy 111.76 35.56))
     (stroke (width 0) (type default) (color 0 0 0 0))
   )
@@
       (effects (font (size 1.27 1.27)) hide)
     )
-    (pin "1")
-  )
-  (symbol (lib_id "Connector:TestPoint") (at 111.76 35.56 0) (unit 1)
-    (in_bom yes) (on_board yes)
-    (property "Reference" "TP9" (id 0) (at 111.76 29.21 0))
-    (property "Value" "TestPoint" (id 1) (at 111.76 25.4 90)
-      (effects (font (size 1.27 1.27)) hide)
-    )
-    (property "Footprint" "TestPoint:TestPoint_Pad_D1.5mm" (id 2) (at 116.84 35.56 0)
-      (effects (font (size 1.27 1.27)) hide)
-    )
-    (property "Datasheet" "~" (id 3) (at 116.84 35.56 0)
-      (effects (font (size 1.27 1.27)) hide)
-    )
-    (property "DNP" "TRUE" (id 4) (at 111.76 35.56 0)
-      (effects (font (size 1.27 1.27)) hide)
-    )
