File: RF-PA-sheet.kicad_sch (KiCad schematic)
At the start: 42 parts, among them J7 SMA_F, J8 U.fl, U10 MHW720A, U14 PSA4-5043 (SPF5043Z), U17 B39431B3710U410

Commit message: SMA LCSC code changed to straight vertical (C496549)
Parts:
- J7: LCSC C411575 -> C496549
Changed lines of the file:
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@@
       (effects (font (size 1.27 1.27)) hide)
     )
-    (property "LCSC" "C411575" (at 24.13 121.92 0)
+    (property "LCSC" "C496549" (at 24.13 121.92 0)
       (effects (font (size 1.27 1.27)) hide)
     )

Commit message: RF capacitor value adjustments based on Tatus lab session 2023-07-12, LCSC codes updated accordingly
Parts:
- C100: value 5p6 -> 8p2; LCSC C519994 -> C519996
- C102, C65: value 5p6 -> 6p8; LCSC C519994 -> C519942
Changed lines of the file:
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@@
       (effects (font (size 1.27 1.27)) (justify left))
     )
-    (property "Value" "5p6" (at 59.4868 123.317 0)
+    (property "Value" "6p8" (at 59.4868 123.317 0)
       (effects (font (size 1.27 1.27)) (justify left))
     )
@@
       (effects (font (size 1.27 1.27)) hide)
     )
-    (property "LCSC" "C519994" (at 57.15 124.46 0)
+    (property "LCSC" "C519942" (at 57.15 124.46 0)
       (effects (font (size 1.27 1.27)) hide)
     )
@@
       (effects (font (size 1.27 1.27)) (justify left))
     )
-    (property "Value" "5p6" (at 95.0468 123.317 0)
+    (property "Value" "8p2" (at 95.0468 123.317 0)
       (effects (font (size 1.27 1.27)) (justify left))
     )
@@
       (effects (font (size 1.27 1.27)) hide)
     )
-    (property "LCSC" "C519994" (at 92.71 124.46 0)
+    (property "LCSC" "C519996" (at 92.71 124.46 0)
       (effects (font (size 1.27 1.27)) hide)
     )
@@
       (effects (font (size 1.27 1.27)) (justify left))
     )
-    (property "Value" "5p6" (at 105.2068 123.317 0)
+    (property "Value" "6p8" (at 105.2068 123.317 0)
       (effects (font (size 1.27 1.27)) (justify left))
     )
@@
       (effects (font (size 1.27 1.27)) hide)
     )
-    (property "LCSC" "C519994" (at 102.87 124.46 0)
-      (effects (font (size 1.27 1.27)) hide)
-    )
+    (property "LCSC" "C519942" (at 102.87 124.46 0)
+      (effects (font (size 1.27 1.27)) hide)
+    )

Commit message: PA DC supply to be filled zone on both BOT&TOP and changed U17,U10 footprints to be of SMD type
Connections:
- net 12V_PA_SUPPLY_FILTERED: now reaches C60.1, C61.1, C62.1, C71.1, L6.2, TP12.1, U10.3 (Vs2)
Changed lines of the file:
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@@
+    )
+  )
+  (global_label "12V_PA_SUPPLY_FILTERED" (shape input) (at 156.21 62.23 0) (fields_autoplaced)
+    (effects (font (size 1.5 1.5) (thickness 0.3) bold) (justify left))
+    (property "Intersheetrefs" "${INTERSHEET_REFS}" (at 188.454 62.23 0)
+      (effects (font (size 1.5 1.5) (thickness 0.3) bold) (justify left) hide)
     )
   )

Commit message: fixed majority of DRC errors
Parts:
- NT2: value 4,5mm+ -> 2,5mm
Other:
- note removed: "+: 5mm tuning tolerance"
Changed lines of the file:
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@@
     (effects (font (size 2.0066 2.0066) (thickness 0.4013) bold) (justify right bottom))
-  )
-  (text "+: 5mm \ntuning tolerance" (at 77.47 135.89 0)
-    (effects (font (size 0.9906 0.9906)) (justify left bottom))
   )
   (text "pin\ndiode" (at 127 116.84 0)
@@
       (effects (font (size 1.27 1.27)) (justify left))
     )
-    (property "Value" "4,5mm+" (at 76.0476 129.413 90)
-      (effects (font (size 1.27 1.27)) (justify left))
-    )
+    (property "Value" "2,5mm" (at 76.0476 129.413 90)
+      (effects (font (size 1.27 1.27)) (justify left))
+    )

Commit message: widened U14 GND pad, new footprint added to NPR library
Parts:
- U14: footprint Package_TO_SOT_SMD:SOT-343_SC-70-4_Handsoldering -> NPR:SOT-343_SC-70-4-widepad_Handsoldering
Changed lines of the file:
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@@
       (effects (font (size 1.27 1.27)))
     )
-    (property "Footprint" "Package_TO_SOT_SMD:SOT-343_SC-70-4_Handsoldering" (at 191.77 121.92 0)
+    (property "Footprint" "NPR:SOT-343_SC-70-4-widepad_Handsoldering" (at 191.77 121.92 0)
       (effects (font (size 1.27 1.27)) hide)
     )

Commit message: added LNA led, adjusted LED resistor for 12V output
Parts:
- NT2: footprint NetTie:NetTie-2_SMD_Pad0.5mm -> NPR:NetTie-2_longer_SMD_Pad0.5mm
Changed lines of the file:
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@@
       (effects (font (size 1.27 1.27)) (justify left))
     )
-    (property "Footprint" "NetTie:NetTie-2_SMD_Pad0.5mm" (at 74.93 128.27 0)
+    (property "Footprint" "NPR:NetTie-2_longer_SMD_Pad0.5mm" (at 74.93 128.27 0)
       (effects (font (size 1.27 1.27)) hide)
     )
