File: RF-PA-sheet.kicad_sch (KiCad schematic)
At the start: 42 parts, among them J7 SMA_F, J8 U.fl, U10 MHW720A, U14 PSA4-5043 (SPF5043Z), U17 B39431B3710U410

Commit message: replace out-of-stock-LCSC codes with available ones
Parts:
- C45, C46: LCSC C400096 -> C597259
- C47, C69, C99: LCSC C519994 -> C513555
- C62: LCSC C2887271 -> C125977
Changed lines of the file:
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@@
 			)
 		)
-		(property "LCSC" "C2887271"
+		(property "LCSC" "C125977"
 			(at 137.16 76.2 0)
 			(effects
@@
 			)
 		)
-		(property "Datasheet" " ~"
+		(property "Datasheet" "~"
 			(at 24.13 121.92 0)
 			(effects
@@
 			)
 		)
-		(property "LCSC" "C400096"
+		(property "LCSC" "C597259"
 			(at 43.18 121.92 0)
 			(effects
@@
 			)
 		)
-		(property "LCSC" "C519994"
+		(property "LCSC" "C513555"
 			(at 140.97 124.46 0)
 			(effects
@@
 			)
 		)
-		(property "LCSC" "C400096"
+		(property "LCSC" "C597259"
 			(at 114.3 121.92 0)
 			(effects
@@
 			)
 		)
-		(property "LCSC" "C519994"
+		(property "LCSC" "C513555"
 			(at 120.65 129.54 0)
 			(effects
@@
 			)
 		)
-		(property "LCSC" "C519994"
+		(property "LCSC" "C513555"
 			(at 49.53 124.46 0)
 			(effects
@@
 			)
 		)
-		(property "Datasheet" " ~"
+		(property "Datasheet" "~"
 			(at 226.06 129.54 0)
 			(effects
